File: 4x4_rotary_macropad.kicad_sch (KiCad schematic)
At the start: 81 parts, among them J1 Conn_01x04_Pin, J2 Conn_01x04_Socket, SW1 SW_Push, SW10 SW_Push, SW11 SW_Push, SW12 SW_Push, SW13 SW_Push, SW14 SW_Push, SW15 SW_Push, SW16 SW_Push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

Commit message: Fixed JLCPCB constraints errors
Parts:
- H1, H2, H3, H4, H5, H6: footprint kbd:M2_HOLE_v3 -> MountingHole:MountingHole_2.2mm_M2
Changed lines of the file:
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@@
       (effects (font (size 1.27 1.27)) (justify left))
     )
-    (property "Footprint" "kbd:M2_HOLE_v3" (at 153.035 173.355 0)
+    (property "Footprint" "MountingHole:MountingHole_2.2mm_M2" (at 153.035 173.355 0)
       (effects (font (size 1.27 1.27)) hide)
     )
@@
       (effects (font (size 1.27 1.27)) (justify left))
     )
-    (property "Footprint" "kbd:M2_HOLE_v3" (at 161.925 165.1 0)
+    (property "Footprint" "MountingHole:MountingHole_2.2mm_M2" (at 161.925 165.1 0)
       (effects (font (size 1.27 1.27)) hide)
     )
@@
       (effects (font (size 1.27 1.27)) (justify left))
     )
-    (property "Footprint" "kbd:M2_HOLE_v3" (at 161.925 181.61 0)
+    (property "Footprint" "MountingHole:MountingHole_2.2mm_M2" (at 161.925 181.61 0)
       (effects (font (size 1.27 1.27)) hide)
     )
@@
       (effects (font (size 1.27 1.27)) (justify left))
     )
-    (property "Footprint" "kbd:M2_HOLE_v3" (at 153.035 181.61 0)
+    (property "Footprint" "MountingHole:MountingHole_2.2mm_M2" (at 153.035 181.61 0)
       (effects (font (size 1.27 1.27)) hide)
     )
@@
       (effects (font (size 1.27 1.27)) (justify left))
     )
-    (property "Footprint" "kbd:M2_HOLE_v3" (at 161.925 173.355 0)
+    (property "Footprint" "MountingHole:MountingHole_2.2mm_M2" (at 161.925 173.355 0)
       (effects (font (size 1.27 1.27)) hide)
     )
@@
       (effects (font (size 1.27 1.27)) (justify left))
     )
-    (property "Footprint" "kbd:M2_HOLE_v3" (at 153.035 165.1 0)
-      (effects (font (size 1.27 1.27)) hide)
-    )
+    (property "Footprint" "MountingHole:MountingHole_2.2mm_M2" (at 153.035 165.1 0)
+      (effects (font (size 1.27 1.27)) hide)
+    )

Commit message: Added missing libraries
Parts:
- removed H5, H6: MountingHole, MountingHole:MountingHole_2.2mm_M2, symbol Mechanical:MountingHole
- removed J1: Conn_01x04_Pin, Connector_Hirose:Hirose_DF13-04P-1.25DS_1x04_P1.25mm_Horizontal, symbol Connector:Conn_01x04_Pin
- removed OLED1: OLED, KiCad-SSD1306-0.91-OLED-4pin-128x32:SSD1306-0.91-OLED-4pin-128x32, symbol utils:OLED
- U1: footprint MCU_RaspberryPi_and_Boards:RPi_Pico_SMD_TH -> cherry_with_keycap:RPi_Pico_SMD_TH
Other:
- moved on the sheet: H1, H2, H3, H4, J2
